File: hardware/_saved_main_pcb.sch (KiCad schematic (older format))
At the start: 39 parts

Commit message: updated schematic, LTC4001 wired
Parts:
- removed J?: AudioStereo, symbol Conn_01x03
- added J?: Headphone PJ325, symbol Audio-Jack-3_2Switches
- added J?: AudioIn, symbol Audio-Jack-3
- L?: value 150nH -> 1500nH
- R? (x2): value 300 -> 470
Connections:
- net +3V3: no longer R?.2, R?.2, R?.2
- net VCC: now also C?.1, R?.2, R?.2, R?.2, U?.8 (PVIN), U?.9 (VINSENSE)
Other:
- note added: "capacitor leads should\nbe kept as short as possible\nbetween PGND and PVIN"
- note added: "low core losses"
Changed lines of the file:
@@
-$EndComp
-$Comp
-L Conn_01x03 J?
-U 1 1 5A559762
-P 10950 4300
-F 0 "J?" H 10950 4500 50  0000 C CNN
-F 1 "AudioStereo" H 10950 4100 50  0000 C CNN
-F 2 "" H 10950 4300 50  0001 C CNN
-F 3 "" H 10950 4300 50  0001 C CNN
-	1    10950 4300
-	1    0    0    -1
 $EndComp
 $Comp
@@
 P 2600 3400
 F 0 "L?" H 2630 3440 50  0000 L CNN
-F 1 "150nH" H 2630 3360 50  0000 L CNN
+F 1 "1500nH" H 2630 3360 50  0000 L CNN
 F 2 "" H 2600 3400 50  0001 C CNN
 F 3 "" H 2600 3400 50  0001 C CNN
@@
 P 4800 3650
 F 0 "R?" H 4830 3670 50  0000 L CNN
-F 1 "300" H 4830 3610 50  0000 L CNN
+F 1 "470" H 4830 3610 50  0000 L CNN
 F 2 "" H 4800 3650 50  0001 C CNN
 F 3 "" H 4800 3650 50  0001 C CNN
@@
 P 5200 3650
 F 0 "R?" H 5230 3670 50  0000 L CNN
-F 1 "300" H 5230 3610 50  0000 L CNN
+F 1 "470" H 5230 3610 50  0000 L CNN
 F 2 "" H 5200 3650 50  0001 C CNN
 F 3 "" H 5200 3650 50  0001 C CNN
@@
 	5200 3850 5200 3750
 Wire Wire Line
-	5200 3450 5200 3550
-Wire Wire Line
-	4800 3450 4800 3550
+	4800 3350 4800 3550
 Text GLabel 4400 4350 0    39   Input ~ 0
 ~CHRG
@@
 	4800 4650 5200 4650
 Connection ~ 5000 4650
-$Comp
-L +3V3 #PWR?
-U 1 1 5A5BC966
-P 5000 3450
-F 0 "#PWR?" H 5000 3300 50  0001 C CNN
-F 1 "+3V3" H 5000 3590 50  0000 C CNN
-F 2 "" H 5000 3450 50  0001 C CNN
-F 3 "" H 5000 3450 50  0001 C CNN
-	1    5000 3450
-	1    0    0    -1
-$EndComp
-Wire Wire Line
-	4450 3450 5200 3450
-Connection ~ 5000 3450
 $Comp
 L R_Small R?
@@
 Connection ~ 3800 3400
 Wire Wire Line
-	3800 3500 3800 3400
+	3800 3300 3800 3500
 Wire Wire Line
 	3100 3550 3100 3300
@@
 	1    0    0    -1
 $EndComp
+Wire Wire Line
+	4450 3450 5200 3450
+Wire Wire Line
+	5200 3450 5200 3550
+$Comp
+L VCC #PWR?
+U 1 1 5A5E10ED
+P 4800 3350
+F 0 "#PWR?" H 4800 3200 50  0001 C CNN
+F 1 "VCC" H 4800 3500 50  0000 C CNN
+F 2 "" H 4800 3350 50  0001 C CNN
+F 3 "" H 4800 3350 50  0001 C CNN
+	1    4800 3350
+	1    0    0    -1
+$EndComp
+$Comp
+L VCC #PWR?
+U 1 1 5A5E18B8
+P 3800 3300
+F 0 "#PWR?" H 3800 3150 50  0001 C CNN
+F 1 "VCC" H 3800 3450 50  0000 C CNN
+F 2 "" H 3800 3300 50  0001 C CNN
+F 3 "" H 3800 3300 50  0001 C CNN
+	1    3800 3300
+	1    0    0    -1
+$EndComp
+Text Notes 2350 3350 0    39   ~ 0
+low core losses
+Text Notes 3450 3500 0    39   ~ 0
+capacitor leads should\nbe kept as short as possible\nbetween PGND and PVIN
+$Comp
+L Audio-Jack-3_2Switches J?
+U 1 1 5A6346F1
+P 10850 6050
+F 0 "J?" H 10850 6340 50  0000 C CNN
+F 1 "Headphone PJ325" H 10700 5850 50  0000 L CNN
+F 2 "" H 11100 6150 50  0001 C CNN
+F 3 "" H 11100 6150 50  0001 C CNN
+	1    10850 6050
+	-1   0    0    1
+$EndComp
+$Comp
+L Audio-Jack-3 J?
+U 1 1 5A6347BA
+P 10850 4550
+F 0 "J?" H 10800 4725 50  0000 C CNN
+F 1 "AudioIn" H 10950 4480 50  0000 C CNN
+F 2 "" H 11100 4650 50  0001 C CNN
+F 3 "" H 11100 4650 50  0001 C CNN
+	1    10850 4550
+	-1   0    0    1
+$EndComp
 $EndSCHEMATC
